Commit message: waffleの3dlidar変更

File: turtlebot3_gazebo/urdf/turtlebot3_waffle.urdf (robot description, URDF)
Before this commit: robot turtlebot3_waffle, 13 links, 12 joints
Links:
- link base_scan: mass 0.114 -> 0.2; geometry collision cylinder length=0.06 radius=0.055; visual cylinder length=0.06 radius=0.055

Commit message: 一部だけ色付けにした

File: turtlebot3_gazebo/urdf/turtlebot3_waffle.urdf (robot description, URDF)
Before this commit: robot turtlebot3_waffle, 13 links, 12 joints
Links:
- link base_link: geometry collision box size=0.266 0.266 0.094; visual box size=0.20 0.20 0.05
- link camera_link: geometry collision box size=0.012 0.132 0.020; visual mesh filename=model://turtlebot3_common/meshes/r200.dae
- link caster_back_left_link: geometry collision box size=0.030 0.009 0.020; visual cylinder length=0.018 radius=0.009
- link caster_back_right_link: geometry collision box size=0.030 0.009 0.020; visual cylinder length=0.018 radius=0.009
- link wheel_left_link: geometry collision cylinder length=0.018 radius=0.033; visual mesh filename=model://turtlebot3_common/meshes/tire.dae scale=0.001 0.001 0.001
- link wheel_right_link: geometry collision cylinder length=0.018 radius=0.033; visual mesh filename=model://turtlebot3_common/meshes/tire.dae scale=0.001 0.001 0.001
Joints:
- joint scan_joint: origin xyz=-0.064 0 0.122 rpy=0 0 0 -> xyz=-0.064 0 0.5 rpy=0 0 0

Commit message: gazeboのbase_linkに修正

File: turtlebot3_gazebo/urdf/turtlebot3_waffle.urdf (robot description, URDF)
Before this commit: robot turtlebot3_waffle, 13 links, 12 joints
Links:
- link base_link: geometry collision box size=0.266 0.266 0.094; visual mesh filename=file:///home/miyake/ros2_ws/src/turtlebot3_gazebo/turtlebot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 scale=0.001 0.001 0.001

Commit message: turtlebot3のパス修正

File: turtlebot3_gazebo/urdf/turtlebot3_waffle.urdf (robot description, URDF)
Before this commit: robot turtlebot3_waffle, 13 links, 12 joints
Links:
- link base_link: geometry collision box size=0.266 0.266 0.094; visual mesh filename=model://turtlebot3_common/meshes/waffle_base.dae scale=0.001 0.001 0.001
